File: Схема осцилографа/1/1.kicad_pcb (KiCad board)
At the start: 2 copper layers, 36 parts, among them U1 LF50_TO252, U2 LM4562

Commit message: Add run only monochrome command
Connections:
- D11 pad 15: unconnected-(D11-XTAL1/CLKN-Pad15) -> GND
Routing:
- net GND: track 400.3 -> 404.9 mm
