File: Схема осцилографа/1/1.kicad_sch (KiCad schematic)
At the start: 36 parts, among them U1 LF50_TO252, U2 LM4562

Commit message: Add run only monochrome command
Connections:
- net GND: now also D11.15 (XTAL1/CLKN)
Changed lines of the file:
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@@
   (junction (at 234.95 80.01) (diameter 0) (color 0 0 0 0)
   )
+  (junction (at 199.39 90.17) (diameter 0) (color 0 0 0 0)
+  )
   (junction (at 212.09 62.23) (diameter 0) (color 0 0 0 0)
   )
@@
     (stroke (width 0) (type default))
   )
+  (wire (pts (xy 199.39 90.17) (xy 204.47 90.17))
+    (stroke (width 0) (type default))
+  )
   (wire (pts (xy 234.95 90.17) (xy 234.95 88.9))
     (stroke (width 0) (type default))
@@
     (stroke (width 0) (type default))
   )
-  (wire (pts (xy 190.5 90.17) (xy 204.47 90.17))
+  (wire (pts (xy 190.5 90.17) (xy 199.39 90.17))
     (stroke (width 0) (type default))
   )
@@
     (stroke (width 0) (type default))
   )
+  (wire (pts (xy 176.53 92.71) (xy 199.39 92.71))
+    (stroke (width 0) (type default))
+  )
   (wire (pts (xy 194.31 50.8) (xy 194.31 53.34))
     (stroke (width 0) (type default))
@@
     (stroke (width 0) (type default))
   )
+  (wire (pts (xy 199.39 92.71) (xy 199.39 90.17))
+    (stroke (width 0) (type default))
+  )
